Commit message: 2023.5.25_pinocchio合并

File: franka_description/robots/panda/panda_withHand.urdf (robot description, URDF)
Before this commit: robot panda, 22 links, 21 joints
Links:
- added link world
- link panda_hand: mass None -> 0.73
- link panda_hand_sc: geometry 
- link panda_leftfinger: mass None -> 0.015
- link panda_link0: mass None -> 0.629769
- link panda_link0_sc: geometry 
- link panda_link1: mass None -> 4.970684
- link panda_link1_sc: geometry 
- link panda_link2: mass None -> 0.646926
- link panda_link2_sc: geometry 
- link panda_link3: mass None -> 3.228604
- link panda_link3_sc: geometry 
- link panda_link4: mass None -> 3.587895
- link panda_link4_sc: geometry 
- link panda_link5: mass None -> 1.225946
- link panda_link5_sc: geometry 
- link panda_link6: mass None -> 1.666555
- link panda_link6_sc: geometry 
- link panda_link7: mass None -> 0.735522
- link panda_link7_sc: geometry 
- link panda_rightfinger: mass None -> 0.015
Joints:
- added joint world_joint: type fixed, parent world, child panda_link0, origin xyz=0 0 0 rpy=0 0 0

File: franka_description/robots/panda/panda_withoutHand.urdf (robot description, URDF)
Before this commit: robot panda, 17 links, 16 joints
Links:
- added link world
- link panda_link0: mass None -> 0.629769
- link panda_link0_sc: geometry 
- link panda_link1: mass None -> 4.970684
- link panda_link1_sc: geometry 
- link panda_link2: mass None -> 0.646926
- link panda_link2_sc: geometry 
- link panda_link3: mass None -> 3.228604
- link panda_link3_sc: geometry 
- link panda_link4: mass None -> 3.587895
- link panda_link4_sc: geometry 
- link panda_link5: mass None -> 1.225946
- link panda_link5_sc: geometry 
- link panda_link6: mass None -> 1.666555
- link panda_link6_sc: geometry 
- link panda_link7: mass None -> 0.735522
- link panda_link7_sc: geometry 
Joints:
- added joint world_joint: type fixed, parent world, child panda_link0, origin xyz=0 0 0 rpy=0 0 0
